File: cpu6502/mem_conn.kicad_sch (KiCad schematic)
At the start: 13 parts, among them J3 Conn_02x21_Odd_Even, U7 ATF22V10C, U8 28C256, U9 74LS00

Commit message: Moved devices around and size reduced board.
Parts:
- removed TP1, TP2, TP3: TestPoint, TestPoint:TestPoint_Pad_2.0x2.0mm, symbol Connector:TestPoint
- added J4, J5: Conn_01x02, Connector_PinHeader_2.54mm:PinHeader_1x02_P2.54mm_Vertical, symbol Connector_Generic:Conn_01x02
- added R7: 10.5K, Resistor_THT:R_Axial_DIN0207_L6.3mm_D2.5mm_P10.16mm_Horizontal, symbol Device:R
Connections:
- net +5V: now also J4.1 (Pin_1), R7.2; no longer U7.1 (I/CLK), U9.10, U9.12, U9.13, U9.9
- net B_A10: now also U7.9 (I8); no longer U7.11 (I10)
- net B_A11: now also U7.7 (I6); no longer U7.10 (I9)
- net B_A12: now also U7.11 (I10); no longer U7.9 (I8)
- net B_A13: now also U7.13 (I11); no longer U7.8 (I7)
- net B_A14: now also U7.10 (I9); no longer U7.7 (I6)
- net B_A15: now also U7.8 (I7); no longer U7.6 (I5)
- net B_A8: now also U7.5 (I4)
- net B_A9: now also U7.6 (I5); no longer U7.13 (I11)
- net ECLK: now also U9.13
- net GND: now also J4.2 (Pin_2), J5.2 (Pin_2)
- net ~{BD_EN}: now also U7.14 (IO10), U9.10, U9.9; no longer U7.5 (I4)
- net ~{BUS_EN}: now also U9.11; no longer U7.14 (IO10)
- net at U9.8: now also U9.12
- new net 32Kn: J5.1 (Pin_1), R7.1, U7.1 (I/CLK)
- no-connect marks 2 -> 0
Other:
- note added: "1 -> 32K ROM 0 -> 8K ROM"
- note added: "BD_ENn ECLK BUS_EN 0 0 1 -> tristate 0 1 0 -> driven 1 0 1 -> tristate 1 1 1 -> tristate"
- note added: "IRQ0n IRQ1n IRQn 0 0 0 0 1 0 1 0 0 1 1 1"
- moved on the sheet: U9C, U9D, U9E

Commit message: Updated to as built.
Parts:
- added R?: 10.5K, Resistor_THT:R_Axial_DIN0207_L6.3mm_D2.5mm_P10.16mm_Horizontal, symbol Device:R
- C10: value 10 uF -> 47 uF
- R6: value 1K -> 3.3K
Connections:
- net +5V: now also R?.2
- net ~{B_WR}: no longer U8.27 (~{WE})
- new net: R?.1, U8.27 (~{WE})
Changed lines of the file:
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@@
 (kicad_sch (version 20211123) (generator eeschema)
   (paper "A4")
+  (junction (at 40.005 161.925) (diameter 0) (color 0 0 0 0)
+  )
   (junction (at 120.65 156.21) (diameter 0) (color 0 0 0 0)
   )
@@
     (stroke (width 0) (type default) (color 0 0 0 0))
   )
-  (wire (pts (xy 50.8 161.925) (xy 59.69 161.925))
+  (wire (pts (xy 38.1 161.925) (xy 40.005 161.925))
     (stroke (width 0) (type default) (color 0 0 0 0))
   )
@@
     (stroke (width 0) (type default) (color 0 0 0 0))
   )
+  (wire (pts (xy 22.86 161.925) (xy 35.56 161.925))
+    (stroke (width 0) (type default) (color 0 0 0 0))
+  )
   (wire (pts (xy 50.8 144.145) (xy 59.69 144.145))
     (stroke (width 0) (type default) (color 0 0 0 0))
@@
     (stroke (width 0) (type default) (color 0 0 0 0))
   )
+  (wire (pts (xy 40.005 149.225) (xy 40.005 151.765))
+    (stroke (width 0) (type default) (color 0 0 0 0))
+  )
   (wire (pts (xy 50.165 86.995) (xy 56.515 86.995))
     (stroke (width 0) (type default) (color 0 0 0 0))
@@
     (stroke (width 0) (type default) (color 0 0 0 0))
   )
+  (wire (pts (xy 40.005 159.385) (xy 40.005 161.925))
+    (stroke (width 0) (type default) (color 0 0 0 0))
+  )
   (wire (pts (xy 27.94 61.595) (xy 31.115 61.595))
     (stroke (width 0) (type default) (color 0 0 0 0))
@@
   )
   (wire (pts (xy 49.53 36.195) (xy 43.815 36.195))
+    (stroke (width 0) (type default) (color 0 0 0 0))
+  )
+  (wire (pts (xy 40.005 161.925) (xy 59.69 161.925))
     (stroke (width 0) (type default) (color 0 0 0 0))
   )
@@
     (effects (font (size 1.27 1.27)) (justify left bottom))
   )
+  (label "write protect memory" (at 20.32 168.91 0)
+    (effects (font (size 1.27 1.27)) (justify left bottom))
+  )
   (label "B_D5" (at 88.9 133.985 180)
     (effects (font (size 1.27 1.27)) (justify right bottom))
@@
     (effects (font (size 1.27 1.27)) (justify left bottom))
   )
+  (label "Cut trace and pullup to" (at 20.955 166.37 0)
+    (effects (font (size 1.27 1.27)) (justify left bottom))
+  )
   (label "B_A12" (at 50.165 92.075 0)
     (effects (font (size 1.27 1.27)) (justify left bottom))
   )
-  (label "~{B_WR}" (at 50.8 161.925 0)
+  (label "~{B_WR}" (at 22.86 161.925 0)
     (effects (font (size 1.27 1.27)) (justify left bottom))
   )
@@
     (in_bom yes) (on_board yes) (fields_autoplaced)
     (property "Reference" "R6" (id 0) (at 227.33 46.99 90))
-    (property "Value" "1K" (id 1) (at 227.33 49.53 90))
+    (property "Value" "3.3K" (id 1) (at 227.33 49.53 90))
     (property "Footprint" "Resistor_THT:R_Axial_DIN0207_L6.3mm_D2.5mm_P10.16mm_Horizontal" (id 2) (at 227.33 54.483 90)
       (effects (font (size 1.27 1.27)) hide)
@@
     (pin "1")
   )
+  (symbol (lib_id "power:+5V") (at 40.005 149.225 0) (unit 1)
+    (in_bom yes) (on_board yes) (fields_autoplaced)
+    (property "Reference" "#PWR?" (id 0) (at 40.005 153.035 0)
+      (effects (font (size 1.27 1.27)) hide)
+    )
+    (property "Value" "+5V" (id 1) (at 40.005 144.145 0))
+    (property "Footprint" "" (id 2) (at 40.005 149.225 0)
+      (effects (font (size 1.27 1.27)) hide)
+    )
+    (property "Datasheet" "" (id 3) (at 40.005 149.225 0)
+      (effects (font (size 1.27 1.27)) hide)
+    )
+    (pin "1")
+  )
   (symbol (lib_id "power:GND") (at 248.92 125.73 0) (unit 1)
     (in_bom yes) (on_board yes) (fields_autoplaced)
@@
       (effects (font (size 1.27 1.27)) (justify left))
     )
-    (property "Value" "10 uF" (id 1) (at 236.22 34.6709 0)
+    (property "Value" "47 uF" (id 1) (at 236.22 34.6709 0)
       (effects (font (size 1.27 1.27)) (justify left))
     )
@@
       (effects (font (size 1.27 1.27)) hide)
     )
+    (pin "1")
+    (pin "2")
+  )
+  (symbol (lib_id "Device:R") (at 40.005 155.575 180) (unit 1)
+    (in_bom yes) (on_board yes) (fields_autoplaced)
+    (property "Reference" "R?" (id 0) (at 42.545 154.3049 0)
+      (effects (font (size 1.27 1.27)) (justify right))
+    )
+    (property "Value" "10.5K" (id 1) (at 42.545 156.8449 0)
+      (effects (font (size 1.27 1.27)) (justify right))
+    )
+    (property "Footprint" "Resistor_THT:R_Axial_DIN0207_L6.3mm_D2.5mm_P10.16mm_Horizontal" (id 2) (at 41.783 155.575 90)
+      (effects (font (size 1.27 1.27)) hide)
+    )
+    (property "Datasheet" "~" (id 3) (at 40.005 155.575 0)
+      (effects (font (size 1.27 1.27)) hide)
+    )
