File: CPU_TESTER/CPU_TESTER.kicad_pcb (KiCad board)
At the start: 2 copper layers, 161.3 x 101.6 mm, 29 parts, among them J1 Conn_02x21_Odd_Even, J2 Conn_02x21_Odd_Even, J3 Conn_02x21_Odd_Even, J4 Conn_02x21_Odd_Even, J5 Conn_02x21_Odd_Even, J6 Conn_02x21_Odd_Even, J7 Conn_02x21_Odd_Even, Q1 2N3904, Q2 2N3904, Q3 2N3904

Commit message: CPU tester design
Parts:
- moved R1 65.1 mm to (50.2, 120.7), turned to -90 degrees
- moved A1 24.9 mm to (64.8, 132.7), turned to 90 degrees
- moved C1 3.20 mm to (55.2, 108.6)
- moved R9 0.63 mm to (50.8, 113.7)
Connections:
- A1 pad 10: BD_EN5 -> /IRQ_0
- A1 pad 11: BD_ENM -> /IRQ_1
- A1 pad 12: /IRQ_0 -> /LED_3
- A1 pad 13: /IRQ_1 -> /LED_4
- A1 pad 14: /RST -> /LED_5
- A1 pad 15: unconnected-(A1-Pad15) -> BD_ENM
- A1 pad 19: /12V_MON -> BD_EN5
- A1 pad 20: /LED_0 -> BD_EN4
- A1 pad 21: /LED_1 -> BD_EN3
- A1 pad 22: /LED_2 -> BD_EN2
- A1 pad 23: /LED_3 -> BD_EN1
- A1 pad 24: /LED_4 -> BD_EN0
- A1 pad 25: /LED_5 -> unconnected-(A1-Pad25)
- A1 pad 26: /LED_C -> /12V_MON
- A1 pad 5: BD_EN0 -> /LED_C
- A1 pad 6: BD_EN1 -> /LED_0
- A1 pad 7: BD_EN2 -> /RST
- A1 pad 8: BD_EN3 -> /LED_1
- A1 pad 9: BD_EN4 -> /LED_2
Routing:
- net +5V: track 131.8 -> 82.4 mm
- net BD_ENM: track 161.0 -> 118.4 mm
- net BD_EN4: track 106.3 -> 76.8 mm
- net BD_EN3: track 83.0 -> 53.9 mm, vias 0 -> 1
- net BD_EN5: track 128.4 -> 102.0 mm
- net /LED_3: track 61.5 -> 35.1 mm
- net /LED_4: track 84.4 -> 58.0 mm
- net /LED_5: track 106.2 -> 80.2 mm
- net /IRQ_0: track 60.0 -> 36.3 mm
- net /LED_0: track 15.1 -> 35.0 mm
- net /LED_2: track 37.9 -> 18.1 mm
- net /IRQ_1: track 37.1 -> 19.8 mm
- net /RST: track 15.3 -> 29.5 mm
- net BD_EN2: track 51.6 -> 37.5 mm
- net /LED_C: track 43.5 -> 30.9 mm
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Other:
- board text added: "USB"
